File: hardware/Fidget/Bus.kicad_sch (KiCad schematic)
At the start: 11 parts, among them J10 ADBUS, J11 SIGBUS, J9 ADBUS-EXP, U15 74AHC16373DG, U16 74AHC16373DG, U17 74LVCC3245APWR

Commit message: Added computie-kicad-library and updated to KiCad 7.0
Parts:
- U15, U16: symbol Fidget:74AHC16373DG -> Computie_Transceivers:74AHC16373DG
- U17: symbol Fidget:74LVCC3245APWR -> Computie_Transceivers:74LVCC3245APWR
