File: hardware/Fidget/LevelShifting.kicad_sch (KiCad schematic)
At the start: 19 parts, among them U10 74ALVC16245DG, U11 74ALVC16245DG, U12 74LVC1G14, U13 74ALVC16245DG, U14 74ALVC16245DG, U8 74ALVC16245DG, U9 74ALVC16245DG

Commit message: Sent Rev.1 to production
Other:
- title: (none) -> Fidget
Changed lines of the file:
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@@
 (kicad_sch (version 20211123) (generator eeschema)
   (paper "A4")
+  (title_block
+    (title "Fidget")
+    (rev "1")
+  )
   (junction (at 203.2 22.86) (diameter 0) (color 0 0 0 0)
   )

Commit message: Added computie-kicad-library and updated to KiCad 7.0
Parts:
- U10, U11, U13, U14, U8, U9: symbol Fidget:74ALVC16245DG -> Computie_Transceivers:74ALVC16245DG
